Commit message: change to moveit from source

File: src/iiwa_stack/iiwa_tool_description/urdf/iiwa_tool.urdf.xacro (robot description, xacro)
@@ -1,9 +1,9 @@
 <?xml version="1.0"?>
 <!-- Here we define the robot, we named it "iiwa7_tool" -->
-<robot xmlns:xacro="http://www.ros.org/wiki/xacro" name="iiwa7_tool">
+<robot xmlns:xacro="http://www.ros.org/wiki/xacro" name="iiwa14_tool">
   <!-- Import Rviz colors -->
   <xacro:include filename="$(find iiwa_description)/urdf/materials.xacro" />
   <!--Import the iiwa7 macro -->
-  <xacro:include filename="$(find iiwa_description)/urdf/iiwa7.xacro"/>
+  <xacro:include filename="$(find iiwa_description)/urdf/iiwa14.xacro"/>
   <!--  Arguments for the iiwa7 macro  -->
   <xacro:arg name="hardware_interface" default="PositionJointInterface"/>
@@ -17,15 +17,80 @@
   <link name="world">
     <visual>
-      <origin xyz="-0.45 -0.18 0.16" rpy="1.57 0 1.57"/>
+      <origin xyz="0.635 1.75 -0.66" rpy="1.57 0 1.57"/>
       <geometry>
-	<mesh filename="package://iiwa_tool_description/meshes/collision/work_cell_base.dae"/>
-	<!-- 	<cylinder length="0.1275" radius="0.020"/> -->
+  <mesh filename="package://iiwa_tool_description/meshes/collision/work_cell_revised.dae"/>
+  <!--  <cylinder length="0.1275" radius="0.020"/> -->
       </geometry>
     </visual>
+            <!-- camera -->
+<visual>
+      <origin xyz="-0.27 0.7 1.17" rpy="0 0 0"/>
+      <geometry>
+  <box size="1 0.5 1"/>
+      </geometry>
+      <material name="Grey"/>
+    </visual>
+                <!-- camera -->
+<collision>
+      <origin xyz="-0.27 0.7 1.17" rpy="0 0 0"/>
+      <geometry>
+  <box size="1 0.5 1"/>
+      </geometry>
+    </collision>
+    <!-- back panel object -->
+<collision>
+      <origin xyz="-1 0.25 0.5" rpy="0 0 0"/>
+      <geometry>
+  <box size="1 4 4"/>
+      </geometry>
+    </collision>
+        <!-- front panel object -->
+<collision>
+      <origin xyz="0.6 0.25 0.5" rpy="0 0 0"/>
+      <geometry>
+  <box size="0.1 4 4"/>
+      </geometry>
+    </collision>
+        <!-- bottom panel object -->
+<collision>
+      <origin xyz="0.08 0.45 0.035" rpy="0 0 0"/>
+      <geometry>
+  <box size="1.3 1.5 0.1"/>
+      </geometry>
+    </collision>
+        <!-- ceiling -->
+<!-- <collision>
+      <origin xyz="0.08 0.45 1.35" rpy="0 0 0"/>
+      <geometry>
+  <box size="1.3 1.5 1"/>
+      </geometry>
+    </collision> -->
+            <!-- side panel object -->
+<collision>
+      <origin xyz="0.14 -0.43 0.5" rpy="0 0 0"/>
+      <geometry>
+  <box size="5 0.4 5"/>
+      </geometry>
+    </collision>
+                <!-- conveyor object -->
+<visual>
+      <origin xyz="0.0 0.7 0.0415" rpy="0 0 0"/>
+      <geometry>
+  <box size="1.5 0.3 .083"/>
+      </geometry>
+      <material name="Grey"/>
+    </visual>
+                <!-- conveyor object -->
+<collision>
+      <origin xyz="0.0 0.7 0.0415" rpy="0 0 0"/>
+      <geometry>
+  <box size="1.5 0.3 .083"/>
+      </geometry>
+    </collision>
     <collision>
-      <origin xyz="-0.45 -0.18 0.16" rpy="1.57 0 1.57"/>
+      <origin xyz="0.635 1.75 -0.69" rpy="1.57 0 1.57"/>
       <geometry>
-	<mesh filename="package://iiwa_tool_description/meshes/collision/work_cell_base.dae"/>
-	<!-- 	<cylinder length="0.1275" radius="0.020"/> -->
+  <mesh filename="package://iiwa_tool_description/meshes/collision/work_cell_revised.dae"/>
+  <!--  <cylinder length="0.1275" radius="0.020"/> -->
       </geometry>
     </collision>
@@ -35,11 +100,11 @@
   </gazebo>
   <!-- Here we insert an iiwa7 robot in the scene, it's origin is just on top of the box previously defined. You can use 0,0,0 if you don't have that. -->
-  <xacro:iiwa7 hardware_interface="$(arg hardware_interface)" robot_name="$(arg robot_name)" parent="world">
-    <origin xyz="0 0 0.84" rpy="0 0 0"/>
-  </xacro:iiwa7>
+  <xacro:iiwa14 hardware_interface="$(arg hardware_interface)" robot_name="$(arg robot_name)" parent="world">
+    <origin xyz="0 0 0" rpy="0 0 0"/>
+  </xacro:iiwa14>
 <!-- Tool properties -->
   <property name="tool_mass" value="0.200" />
   <property name="tool_joint_offset" value="0.00 0.00 0.00" />
-  <property name="tool_link_offset" value="0.00 0.00 0.1275" />
+  <property name="tool_link_offset" value="0.00 0.00 0.23" />
   <!--  Here we define a dummy joint between the tip of the iiwa7 and the base of the tool.
   There is no offset between the two, that means the tool is attached at the robot flange. -->
@@ -47,5 +112,5 @@
     <parent link="iiwa_link_ee" />
     <child link = "tool_link" />
-    <origin xyz="${tool_joint_offset}" rpy="0 ${PI/2.0} 0" />
+    <origin xyz="${tool_joint_offset}" rpy="0 0 0" />
   </joint>
   <!-- Here we define the geometry of the tool. We designed the tool ourselves, so we have a mesh file that represents it.
@@ -53,16 +118,16 @@
   <link name="tool_link">
     <visual>
-      <origin xyz="0 0 0" rpy="0 0 0"/>
+      <origin xyz="0 0 0.12" rpy="0 0 0"/>
       <geometry>
-	<mesh filename="package://iiwa_tool_description/meshes/visual/tool.stl"/>
-	<!-- 	<cylinder length="0.1275" radius="0.020"/> -->
+  <!-- <mesh filename="package://iiwa_tool_description/meshes/visual/tool.dae"/> -->
+  <cylinder length="0.24" radius="0.08"/>
       </geometry>
       <material name="Grey"/>
     </visual>
     <collision>
-      <origin xyz="0 0 0" rpy="0 0 0"/>
+      <origin xyz="0 0 0.115" rpy="0 0 0"/>
       <geometry>
-	<mesh filename="package://iiwa_tool_description/meshes/visual/tool.stl"/>
-	<!-- 	<cylinder length="0.1275" radius="0.020"/> -->
+  <!-- <mesh filename="package://iiwa_tool_description/meshes/visual/tool.dae"/> -->
+  <cylinder length="0.23" radius="0.07"/>
       </geometry>
       <material name="Grey"/>

Commit message: added functionality to save/load trajectories

File: src/iiwa_stack/iiwa_tool_description/urdf/iiwa_tool.urdf.xacro (robot description, xacro)
@@ -1,64 +1,64 @@
-<?xml version="1.0"?>
+<?xml version="1.0" encoding="UTF-8"?>
 <!-- Here we define the robot, we named it "iiwa7_tool" -->
 <robot xmlns:xacro="http://www.ros.org/wiki/xacro" name="iiwa14_tool">
-  <!-- Import Rviz colors -->
-  <xacro:include filename="$(find iiwa_description)/urdf/materials.xacro" />
-  <!--Import the iiwa7 macro -->
-  <xacro:include filename="$(find iiwa_description)/urdf/iiwa14.xacro"/>
-  <!--  Arguments for the iiwa7 macro  -->
-  <xacro:arg name="hardware_interface" default="PositionJointInterface"/>
-  <xacro:arg name="robot_name" default="iiwa"/>
-  <!--  Define the origin of your 3D space
+   <!-- Import Rviz colors -->
+   <xacro:include filename="$(find iiwa_description)/urdf/materials.xacro" />
+   <!--Import the iiwa7 macro -->
+   <xacro:include filename="$(find iiwa_description)/urdf/iiwa14.xacro" />
+   <!--  Arguments for the iiwa7 macro  -->
+   <xacro:arg name="hardware_interface" default="PositionJointInterface" />
+   <xacro:arg name="robot_name" default="iiwa" />
+   <!--  Define the origin of your 3D space
   Here we define a box lying at 0,0,0 with some dimensions, in reality our robot is place on top of a metal cart with those dimensions.
   This will include the cart in the scene and avoid the robot to hit it when using MoveIt!
   If you don't want to have that you can define a basic world link (see commented lines)
   -->
-  <!--     <link name="world"/> -->
-  <link name="world">
-    <visual>
-      <origin xyz="0.635 1.75 -0.66" rpy="1.57 0 1.57"/>
-      <geometry>
-  <mesh filename="package://iiwa_tool_description/meshes/collision/work_cell_revised.dae"/>
-  <!--  <cylinder length="0.1275" radius="0.020"/> -->
-      </geometry>
-    </visual>
-            <!-- camera -->
-<visual>
-      <origin xyz="-0.27 0.7 1.17" rpy="0 0 0"/>
-      <geometry>
-  <box size="1 0.5 1"/>
-      </geometry>
-      <material name="Grey"/>
-    </visual>
-                <!-- camera -->
-<collision>
-      <origin xyz="-0.27 0.7 1.17" rpy="0 0 0"/>
-      <geometry>
-  <box size="1 0.5 1"/>
-      </geometry>
-    </collision>
-    <!-- back panel object -->
-<collision>
-      <origin xyz="-1 0.25 0.5" rpy="0 0 0"/>
-      <geometry>
-  <box size="1 4 4"/>
-      </geometry>
-    </collision>
-        <!-- front panel object -->
-<collision>
-      <origin xyz="0.6 0.25 0.5" rpy="0 0 0"/>
-      <geometry>
-  <box size="0.1 4 4"/>
-      </geometry>
-    </collision>
-        <!-- bottom panel object -->
-<collision>
-      <origin xyz="0.08 0.45 0.035" rpy="0 0 0"/>
-      <geometry>
-  <box size="1.3 1.5 0.1"/>
-      </geometry>
-    </collision>
-        <!-- ceiling -->
-<!-- <collision>
+   <!--     <link name="world"/> -->
+   <link name="world">
+      <visual>
+         <origin xyz="0.635 1.75 -0.66" rpy="1.57 0 1.57" />
+         <geometry>
+            <mesh filename="package://iiwa_tool_description/meshes/collision/work_cell_revised.dae" />
+            <!--  <cylinder length="0.1275" radius="0.020"/> -->
+         </geometry>
+      </visual>
+      <!-- camera visual -->
+      <visual>
+         <origin xyz="-0.27 0.7 1.4" rpy="0 0 0" />
+         <geometry>
+            <box size="1 0.5 1" />
+         </geometry>
+         <material name="Grey" />
+      </visual>
+      <!-- camera collision-->
+      <collision>
+         <origin xyz="-0.27 0.7 1.4" rpy="0 0 0" />
+         <geometry>
+            <box size="1 0.5 1" />
+         </geometry>
+      </collision>
+      <!-- back panel object -->
+      <collision>
+         <origin xyz="-1 0.25 0.5" rpy="0 0 0" />
+         <geometry>
+            <box size="1 4 4" />
+         </geometry>
+      </collision>
+      <!-- front panel object -->
+      <collision>
+         <origin xyz="0.6 0.25 0.5" rpy="0 0 0" />
+         <geometry>
+            <box size="0.1 4 4" />
+         </geometry>
+      </collision>
+      <!-- bottom panel object -->
+      <collision>
+         <origin xyz="0.08 0.75 0.035" rpy="0 0 0" />
+         <geometry>
+            <box size="1.3 2 0.1" />
+         </geometry>
+      </collision>
+      <!-- ceiling -->
+      <!-- <collision>
       <origin xyz="0.08 0.45 1.35" rpy="0 0 0"/>
       <geometry>
@@ -66,79 +66,79 @@
       </geometry>
     </collision> -->
-            <!-- side panel object -->
-<collision>
-      <origin xyz="0.14 -0.43 0.5" rpy="0 0 0"/>
-      <geometry>
-  <box size="5 0.4 5"/>
-      </geometry>
-    </collision>
-                <!-- conveyor object -->
-<visual>
-      <origin xyz="0.0 0.7 0.0415" rpy="0 0 0"/>
-      <geometry>
-  <box size="1.5 0.3 .083"/>
-      </geometry>
-      <material name="Grey"/>
-    </visual>
-                <!-- conveyor object -->
-<collision>
-      <origin xyz="0.0 0.7 0.0415" rpy="0 0 0"/>
-      <geometry>
-  <box size="1.5 0.3 .083"/>
-      </geometry>
-    </collision>
-    <collision>
-      <origin xyz="0.635 1.75 -0.69" rpy="1.57 0 1.57"/>
-      <geometry>
-  <mesh filename="package://iiwa_tool_description/meshes/collision/work_cell_revised.dae"/>
-  <!--  <cylinder length="0.1275" radius="0.020"/> -->
-      </geometry>
-    </collision>
-  </link>
-  <gazebo reference="world">
-    <static>true</static>
-  </gazebo>
-  <!-- Here we insert an iiwa7 robot in the scene, it's origin is just on top of the box previously defined. You can use 0,0,0 if you don't have that. -->
-  <xacro:iiwa14 hardware_interface="$(arg hardware_interface)" robot_name="$(arg robot_name)" parent="world">
-    <origin xyz="0 0 0" rpy="0 0 0"/>
-  </xacro:iiwa14>
-<!-- Tool properties -->
-  <property name="tool_mass" value="0.200" />
-  <property name="tool_joint_offset" value="0.00 0.00 0.00" />
-  <property name="tool_link_offset" value="0.00 0.00 0.23" />
-  <!--  Here we define a dummy joint between the tip of the iiwa7 and the base of the tool.
+      <!-- side panel object -->
+      <collision>
+         <origin xyz="0.14 -0.43 0.5" rpy="0 0 0" />
+         <geometry>
+            <box size="5 0.4 5" />
+         </geometry>
+      </collision>
+      <!-- conveyor object visual -->
+      <visual>
+         <origin xyz="0.0 0.7 0.0415" rpy="0 0 0" />
+         <geometry>
+            <box size="1.2 0.7 .083" />
+         </geometry>
+         <material name="Grey" />
+      </visual>
+      <!-- conveyor object collision -->
+      <collision>
+         <origin xyz="0.0 0.7 0.0415" rpy="0 0 0" />
+         <geometry>
+            <box size="1.2 0.7 .083" />
+         </geometry>
+      </collision>
+      <collision>
+         <origin xyz="0.635 1.75 -0.69" rpy="1.57 0 1.57" />
+         <geometry>
+            <mesh filename="package://iiwa_tool_description/meshes/collision/work_cell_revised.dae" />
+            <!--  <cylinder length="0.1275" radius="0.020"/> -->
+         </geometry>
+      </collision>
+   </link>
+   <gazebo reference="world">
+      <static>true</static>
+   </gazebo>
+   <!-- Here we insert an iiwa7 robot in the scene, it's origin is just on top of the box previously defined. You can use 0,0,0 if you don't have that. -->
+   <xacro:iiwa14 hardware_interface="$(arg hardware_interface)" robot_name="$(arg robot_name)" parent="world">
+      <origin xyz="0 0 0" rpy="0 0 0" />
+   </xacro:iiwa14>
+   <!-- Tool properties -->
+   <property name="tool_mass" value="0.200" />
+   <property name="tool_joint_offset" value="0.00 0.00 0.00" />
+   <property name="tool_link_offset" value="0.00 0.00 0.23" />
+   <!--  Here we define a dummy joint between the tip of the iiwa7 and the base of the tool.
   There is no offset between the two, that means the tool is attached at the robot flange. -->
-  <joint name="tool_joint" type="fixed">
-    <parent link="iiwa_link_ee" />
-    <child link = "tool_link" />
-    <origin xyz="${tool_joint_offset}" rpy="0 0 0" />
-  </joint>
-  <!-- Here we define the geometry of the tool. We designed the tool ourselves, so we have a mesh file that represents it.
+   <joint name="tool_joint" type="fixed">
+      <parent link="iiwa_link_ee" />
+      <child link="tool_link" />
+      <origin xyz="${tool_joint_offset}" rpy="0 0 0" />
+   </joint>
+   <!-- Here we define the geometry of the tool. We designed the tool ourselves, so we have a mesh file that represents it.
   Else, one can define it using a geometric representation that approximate it, like a cylinder (see commented lines) -->
-  <link name="tool_link">
-    <visual>
-      <origin xyz="0 0 0.12" rpy="0 0 0"/>
-      <geometry>
-  <!-- <mesh filename="package://iiwa_tool_description/meshes/visual/tool.dae"/> -->
-  <cylinder length="0.24" radius="0.08"/>
-      </geometry>
-      <material name="Grey"/>
-    </visual>
-    <collision>
-      <origin xyz="0 0 0.115" rpy="0 0 0"/>
-      <geometry>
-  <!-- <mesh filename="package://iiwa_tool_description/meshes/visual/tool.dae"/> -->
-  <cylinder length="0.23" radius="0.07"/>
-      </geometry>
-      <material name="Grey"/>
-    </collision>
-  </link>
-  <!--  Here we define another dummy joint. It is placed at the end of the tool, so we can then attach a frame at its TCP for control -->
-  <joint name="tool_tip_joint" type="fixed">
-    <parent link="tool_link" />
-    <child link = "tool_link_ee" />
-    <origin xyz="${tool_link_offset}" rpy="0 0 0" />
-  </joint>
-  <!--  The TCP frame is here defined -->
-  <link name="tool_link_ee"/>
+   <link name="tool_link">
+      <visual>
+         <origin xyz="0 0 0.12" rpy="0 0 0" />
+         <geometry>
+            <!-- <mesh filename="package://iiwa_tool_description/meshes/visual/tool.dae"/> -->
+            <cylinder length="0.24" radius="0.08" />
+         </geometry>
+         <material name="Grey" />
+      </visual>
+      <collision>
+         <origin xyz="0 0 0.115" rpy="0 0 0" />
+         <geometry>
+            <!-- <mesh filename="package://iiwa_tool_description/meshes/visual/tool.dae"/> -->
+            <cylinder length="0.23" radius="0.07" />
+         </geometry>
+         <material name="Grey" />
+      </collision>
+   </link>
+   <!--  Here we define another dummy joint. It is placed at the end of the tool, so we can then attach a frame at its TCP for control -->
+   <joint name="tool_tip_joint" type="fixed">
+      <parent link="tool_link" />
+      <child link="tool_link_ee" />
+      <origin xyz="${tool_link_offset}" rpy="0 0 0" />
+   </joint>
+   <!--  The TCP frame is here defined -->
+   <link name="tool_link_ee" />
 </robot>

Commit message: changed to map for components

File: src/iiwa_stack/iiwa_tool_description/urdf/iiwa_tool.urdf.xacro (robot description, xacro)
@@ -75,7 +75,7 @@
       <!-- conveyor object visual -->
       <visual>
-         <origin xyz="0.0 0.7 0.0415" rpy="0 0 0" />
+         <origin xyz="0.0 0.7 0.0635" rpy="0 0 0" />
          <geometry>
-            <box size="1.2 0.7 .083" />
+            <box size="1.2 0.7 .127" />
          </geometry>
          <material name="Grey" />
@@ -83,7 +83,7 @@
       <!-- conveyor object collision -->
       <collision>
-         <origin xyz="0.0 0.7 0.0415" rpy="0 0 0" />
+         <origin xyz="0.0 0.7 0.0635" rpy="0 0 0" />
          <geometry>
-            <box size="1.2 0.7 .083" />
+            <box size="1.2 0.7 .127" />
          </geometry>
       </collision>

Commit message: add config.py, hdd rotation

File: src/iiwa_stack/iiwa_tool_description/urdf/iiwa_tool.urdf.xacro (robot description, xacro)
@@ -47,5 +47,5 @@
       <!-- front panel object -->
       <collision>
-         <origin xyz="0.6 0.25 0.5" rpy="0 0 0" />
+         <origin xyz="1 0.25 0.5" rpy="0 0 0" />
          <geometry>
             <box size="0.1 4 4" />

Commit message: fix urdf and extend_trajectory

File: src/iiwa_stack/iiwa_tool_description/urdf/iiwa_tool.urdf.xacro (robot description, xacro)
@@ -17,5 +17,5 @@
    <link name="world">
       <visual>
-         <origin xyz="0.635 1.75 -0.66" rpy="1.57 0 1.57" />
+         <origin xyz="0.635 1.751 -0.687" rpy="1.57 0 1.57" />
          <geometry>
             <mesh filename="package://iiwa_tool_description/meshes/collision/work_cell_revised.dae" />
@@ -25,5 +25,5 @@
       <!-- camera visual -->
       <visual>
-         <origin xyz="-0.27 0.7 1.4" rpy="0 0 0" />
+         <origin xyz="-0.27 0.7 1.33" rpy="0 0 0" />
          <geometry>
             <box size="1 0.5 1" />
@@ -33,5 +33,5 @@
       <!-- camera collision-->
       <collision>
-         <origin xyz="-0.27 0.7 1.4" rpy="0 0 0" />
+         <origin xyz="-0.27 0.7 1.33" rpy="0 0 0" />
          <geometry>
             <box size="1 0.5 1" />
@@ -40,5 +40,5 @@
       <!-- back panel object -->
       <collision>
-         <origin xyz="-1 0.25 0.5" rpy="0 0 0" />
+         <origin xyz="-0.94 0.25 0.5" rpy="0 0 0" />
          <geometry>
             <box size="1 4 4" />
@@ -47,5 +47,5 @@
       <!-- front panel object -->
       <collision>
-         <origin xyz="1 0.25 0.5" rpy="0 0 0" />
+         <origin xyz="0.7 0.25 0.5" rpy="0 0 0" />
          <geometry>
             <box size="0.1 4 4" />
@@ -54,5 +54,5 @@
       <!-- bottom panel object -->
       <collision>
-         <origin xyz="0.08 0.75 0.035" rpy="0 0 0" />
+         <origin xyz="0.08 0.75 0.03" rpy="0 0 0" />
          <geometry>
             <box size="1.3 2 0.1" />
@@ -75,5 +75,5 @@
       <!-- conveyor object visual -->
       <visual>
-         <origin xyz="0.0 0.7 0.0635" rpy="0 0 0" />
+         <origin xyz="0.0 0.7 0.043" rpy="0 0 0" />
          <geometry>
             <box size="1.2 0.7 .127" />
@@ -83,5 +83,5 @@
       <!-- conveyor object collision -->
       <collision>
-         <origin xyz="0.0 0.7 0.0635" rpy="0 0 0" />
+         <origin xyz="0.0 0.7 0.043" rpy="0 0 0" />
          <geometry>
             <box size="1.2 0.7 .127" />
@@ -104,5 +104,5 @@
    </xacro:iiwa14>
    <!-- Tool properties -->
-   <property name="tool_mass" value="0.200" />
+   <property name="tool_mass" value="1.00" />
    <property name="tool_joint_offset" value="0.00 0.00 0.00" />
    <property name="tool_link_offset" value="0.00 0.00 0.23" />
@@ -121,5 +121,5 @@
          <geometry>
             <!-- <mesh filename="package://iiwa_tool_description/meshes/visual/tool.dae"/> -->
-            <cylinder length="0.24" radius="0.08" />
+            <cylinder length="0.24" radius="0.09" />
          </geometry>
          <material name="Grey" />
@@ -129,5 +129,5 @@
          <geometry>
             <!-- <mesh filename="package://iiwa_tool_description/meshes/visual/tool.dae"/> -->
-            <cylinder length="0.23" radius="0.07" />
+            <cylinder length="0.23" radius="0.09" />
          </geometry>
          <material name="Grey" />
