Commit message: two arms works!!!

File: src/iiwa_stack/iiwa_tool_description/urdf/iiwa_tool.urdf.xacro (robot description, xacro)
@@ -25,5 +25,5 @@
       <!-- camera visual -->
       <visual>
-         <origin xyz="-0.27 0.7 1.33" rpy="0 0 0" />
+         <origin xyz="-0.27 0.7 1.37" rpy="0 0 0" />
          <geometry>
             <box size="1 1.3 1" />
@@ -33,5 +33,5 @@
       <!-- camera collision-->
       <collision>
-         <origin xyz="-0.27 0.7 1.33" rpy="0 0 0" />
+         <origin xyz="-0.27 0.7 1.37" rpy="0 0 0" />
          <geometry>
             <box size="1 1.3 1" />
@@ -67,10 +67,26 @@
     </collision> -->
       <!-- side panel object -->
-      <!-- <collision>
-         <origin xyz="0.14 -0.43 0.5" rpy="0 0 0" />
+      <!-- <visual>
+         <origin xyz="0.14 1.2 0.5" rpy="0 0 0" />
          <geometry>
             <box size="5 0.4 5" />
          </geometry>
-      </collision> -->
+      </visual> -->
+      <!-- tray object visual -->
+      <visual>
+         <origin xyz="0.45 0.05 0.043" rpy="0 0 0" />
+         <geometry>
+            <box size="0.35 0.5 .12" />
+         </geometry>
+         <material name="Grey" />
+      </visual>
+      <!-- tray object collision -->
+      <collision>
+         <origin xyz="0.45 0.05 0.043" rpy="0 0 0" />
+         <geometry>
+            <box size="0.35 0.5 .12" />
+         </geometry>
+         <material name="Grey" />
+      </collision>
       <!-- conveyor object visual -->
       <visual>
@@ -101,10 +117,10 @@
    <!-- Here we insert an iiwa7 robot in the scene, it's origin is just on top of the box previously defined. You can use 0,0,0 if you don't have that. -->
    <xacro:iiwa14 hardware_interface="$(arg hardware_interface)" robot_name="$(arg robot_name)" parent="world">
-      <origin xyz="0 1.5 0" rpy="0 0 0" />
+      <origin xyz="0 0 0" rpy="0 0 0" />
    </xacro:iiwa14>
    <!-- Tool properties -->
    <property name="tool_mass" value="1.00" />
    <property name="tool_joint_offset" value="0.00 0.00 0.00" />
-   <property name="tool_link_offset" value="0.00 0.00 0.23" />
+   <property name="tool_link_offset" value="0.00 0.00 0.25" />
    <!--  Here we define a dummy joint between the tip of the iiwa7 and the base of the tool.
   There is no offset between the two, that means the tool is attached at the robot flange. -->
@@ -121,5 +137,5 @@
          <geometry>
             <!-- <mesh filename="package://iiwa_tool_description/meshes/visual/tool.dae"/> -->
-            <cylinder length="0.24" radius="0.09" />
+            <cylinder length="0.25" radius="0.09" />
          </geometry>
          <material name="Grey" />
@@ -129,5 +145,5 @@
          <geometry>
             <!-- <mesh filename="package://iiwa_tool_description/meshes/visual/tool.dae"/> -->
-            <cylinder length="0.23" radius="0.09" />
+            <cylinder length="0.25" radius="0.09" />
          </geometry>
          <material name="Grey" />

File: src/iiwa_stack/iiwa_tool_description/urdf/iiwa_tool_right.urdf.xacro (robot description, xacro)
@@ -101,5 +101,5 @@
    <!-- Here we insert an iiwa7 robot in the scene, it's origin is just on top of the box previously defined. You can use 0,0,0 if you don't have that. -->
    <xacro:iiwa14 hardware_interface="$(arg hardware_interface)" robot_name="$(arg robot_name)" parent="world">
-      <origin xyz="0 0 0" rpy="0 0 0" />
+      <origin xyz="0 1.5 0" rpy="0 0 0" />
    </xacro:iiwa14>
    <!-- Tool properties -->
@@ -110,5 +110,5 @@
   There is no offset between the two, that means the tool is attached at the robot flange. -->
    <joint name="tool_joint" type="fixed">
-      <parent link="iiwa_link_ee" />
+      <parent link="iiwa2_link_ee" />
       <child link="tool_link" />
       <origin xyz="${tool_joint_offset}" rpy="0 0 0" />

Commit message: spring demo

File: src/iiwa_stack/iiwa_tool_description/urdf/iiwa_tool.urdf.xacro (robot description, xacro)
@@ -38,7 +38,14 @@
          </geometry>
       </collision>
+      <!-- ceiling-->
+      <collision>
+         <origin xyz="-0.27 0.7 1.37" rpy="0 0 0" />
+         <geometry>
+            <box size="6 6 1" />
+         </geometry>
+      </collision>
       <!-- back panel object -->
       <collision>
-         <origin xyz="-0.94 0.25 0.5" rpy="0 0 0" />
+         <origin xyz="-0.99 0.25 0.5" rpy="0 0 0" />
          <geometry>
             <box size="1 4 4" />
@@ -47,5 +54,5 @@
       <!-- front panel object -->
       <collision>
-         <origin xyz="0.7 0.25 0.5" rpy="0 0 0" />
+         <origin xyz="0.9 0.25 0.5" rpy="0 0 0" />
          <geometry>
             <box size="0.1 4 4" />
@@ -54,5 +61,5 @@
       <!-- bottom panel object -->
       <collision>
-         <origin xyz="0.08 0.75 0.03" rpy="0 0 0" />
+         <origin xyz="0.08 0.75 0.01" rpy="0 0 0" />
          <geometry>
             <box size="1.3 2 0.1" />
@@ -75,5 +82,5 @@
       <!-- tray object visual -->
       <visual>
-         <origin xyz="0.45 0.05 0.043" rpy="0 0 0" />
+         <origin xyz="0.45 0.05 0.003" rpy="0 0 0" />
          <geometry>
             <box size="0.35 0.5 .12" />
@@ -83,5 +90,5 @@
       <!-- tray object collision -->
       <collision>
-         <origin xyz="0.45 0.05 0.043" rpy="0 0 0" />
+         <origin xyz="0.45 0.05 0.003" rpy="0 0 0" />
          <geometry>
             <box size="0.35 0.5 .12" />
@@ -89,7 +96,23 @@
          <material name="Grey" />
       </collision>
+            <!-- conveyor motor visual -->
+      <!-- <visual>
+         <origin xyz="-0.25 0.24 0.06" rpy="0 0 0" />
+         <geometry>
+            <box size="0.40 0.20 .14" />
+         </geometry>
+         <material name="Grey" />
+      </visual> -->
+      <!-- conveyor motor collision -->
+      <!-- <collision>
+         <origin xyz="-0.25 0.24 0.06" rpy="0 0 0" />
+         <geometry>
+            <box size="0.40 0.20 .14" />
+         </geometry>
+         <material name="Grey" />
+      </collision> -->
       <!-- conveyor object visual -->
       <visual>
-         <origin xyz="0.0 0.7 0.043" rpy="0 0 0" />
+         <origin xyz="0.0 0.7 0.013" rpy="0 0 0" />
          <geometry>
             <box size="1.2 0.7 .127" />
@@ -97,7 +120,23 @@
          <material name="Grey" />
       </visual>
+            <!-- tray table visual -->
+      <visual>
+         <origin xyz="-0 -0.5 -0.1" rpy="0 0 0" />
+         <geometry>
+            <box size="1.1 0.5 0.7" />
+         </geometry>
+         <material name="Grey" />
+      </visual>
+      <!-- tray table visual -->
+      <collision>
+         <origin xyz="-0 -0.5 -0.1" rpy="0 0 0" />
+         <geometry>
+            <box size="1.1 0.5 0.7" />
+         </geometry>
+         <material name="Grey" />
+      </collision>
       <!-- conveyor object collision -->
       <collision>
-         <origin xyz="0.0 0.7 0.043" rpy="0 0 0" />
+         <origin xyz="0.0 0.7 0.013" rpy="0 0 0" />
          <geometry>
             <box size="1.2 0.7 .127" />

File: src/iiwa_stack/iiwa_tool_description/urdf/iiwa_tool_right.urdf.xacro (robot description, xacro)
@@ -121,5 +121,5 @@
          <geometry>
             <!-- <mesh filename="package://iiwa_tool_description/meshes/visual/tool.dae"/> -->
-            <cylinder length="0.24" radius="0.09" />
+            <cylinder length="0.24" radius="0.06" />
          </geometry>
          <material name="Grey" />
@@ -129,5 +129,5 @@
          <geometry>
             <!-- <mesh filename="package://iiwa_tool_description/meshes/visual/tool.dae"/> -->
-            <cylinder length="0.23" radius="0.09" />
+            <cylinder length="0.23" radius="0.06" />
          </geometry>
          <material name="Grey" />
